File: SinCosEnc-Converter_EP5101-0011.kicad_pcb (KiCad board)
At the start: 2 copper layers, 88 x 61.8 mm, 95 parts, among them J1 Conn_02x05_Top_Bottom, SW1 SW_RCLK, SW2 SW_SG1, SW3 SW_SG0, SW4 SW_ROT, SW5 SW_SF1, SW6 SW_SF0, U1 iC-NV, U2 AM26LS31CDR, U3 AP22652AW6-7, U4 LM66100DCKR, X2 D-SUB-DR-15PCG-AB

Commit message: Last unfinished project state -> ARCHIVED
PCB version v0.9.6 was fully working and successfully tested. Version v0.9.8 was never produced nor tested.
This board is provided as is - unfinished and untested. Productive use is explicitly not recommended! Further rework is required. No support is offered for it. The project will be left as is.
Parts:
- removed MH1: MountingHole_3.2mm_M3_ISO14580, MountingHole:MountingHole_3.2mm_M3_ISO14580
- added G***: LOGO, LOGO, F.Cu at (132.1, 66.6)
- added H1: MountingHole_Pad, MountingHole:MountingHole_3.2mm_M3_DIN965_Pad_TopBottom, F.Cu at (132.1, 61.1)
- C11: value 0.1u -> 100n
- R1: value 215k -> 120k
- moved REF** 7.74 mm to (126.3, 61.2), turned to 90 degrees
- moved C6 1.74 mm to (92.9, 99.4)
Connections:
- J1 pad 8: GNDS -> GND
Routing:
- net GNDS: track 160.6 -> 204.6 mm
- net +5V: track 264.0 -> 279.0 mm
- net GND: track 146.0 -> 139.8 mm, vias 125 -> 147
- net +5V_Sensor: track 96.6 -> 99.9 mm
- net Net-(SW1-B): track 65.2 -> 63.3 mm
- net CON_~{ERR}: track 124.2 -> 123.6 mm
- net (no net): vias 0 -> 1
Other:
- outline, holes or cut-outs redrawn
- board text added: "8 GNDsh"
- board text added: "use Pin 8 of PinHeader for internal shield"
- board text removed: "8 Shield"
