File: SinCosEnc-Converter_EP5101-0011.kicad_sch (KiCad schematic)
At the start: 40 parts, among them U2 AM26LS31CDR, U3 AP22652AW6-7, U4 LM66100DCKR, X2 D-SUB-DR-15PCG-AB

Commit message: Last unfinished project state -> ARCHIVED
PCB version v0.9.6 was fully working and successfully tested. Version v0.9.8 was never produced nor tested.
This board is provided as is - unfinished and untested. Productive use is explicitly not recommended! Further rework is required. No support is offered for it. The project will be left as is.
Parts:
- added H1: MountingHole_Pad, MountingHole:MountingHole_3.2mm_M3_DIN965_Pad_TopBottom, symbol Mechanical:MountingHole_Pad
- C11: value 0.1u -> 100n; LCSC Part (none) -> C14663
- C6, C7: LCSC Part (none) -> C14663
- C8: LCSC Part (none) -> C15849
- C9: LCSC Part (none) -> C91606
- D2, D3, D4, D5, D6, D7: value SD15 -> SD15C
- R1: value 215k -> 120k
Connections:
- net GNDS: now also H1.1
Other:
- note added: "NOTE: ILIM with 120k (R1) = 195 mA max. Output (\sqrt{1.055}{30321/195mA})"
- note removed: "NOTE: ILIM with 215k (R1) = 105 mA max. Output (\sqrt{1.055}{30321/105mA})"
- moved on the sheet: C13, R12
